Commit message: change urdf dof limit, change reward for wow

File: legged_train/resources/robots/wow/urdf/wow.urdf (robot description, URDF)
Before this commit: robot wow1, 11 links, 10 joints
Joints:
- joint left_knee_joint: limit lower=0 upper=1.57 effort=58 velocity=23 -> lower=0 upper=1.1 effort=58 velocity=23
- joint left_pitch_joint: limit lower=-1.57 upper=0.5 effort=58 velocity=23 -> lower=-1 upper=0.5 effort=58 velocity=23
- joint left_roll_joint: limit lower=-0.2 upper=1.5 effort=30 velocity=23 -> lower=-0.2 upper=0.5 effort=30 velocity=23
- joint right_knee_joint: limit lower=-1.57 upper=0 effort=58 velocity=23 -> lower=-1.1 upper=0 effort=58 velocity=23
- joint right_pitch_joint: limit lower=-0.5 upper=1.57 effort=58 velocity=23 -> lower=-0.3 upper=0.3 effort=58 velocity=23
- joint right_roll_joint: limit lower=-1.57 upper=0.2 effort=30 velocity=23 -> lower=-0.5 upper=0.2 effort=30 velocity=23
- joint right_yaw_joint: limit lower=-0.5 upper=0.5 effort=30 velocity=23 -> lower=-0.3 upper=0.3 effort=30 velocity=23

Commit message: can walk solwly

File: legged_train/resources/robots/wow/urdf/wow.urdf (robot description, URDF)
Before this commit: robot wow1, 11 links, 10 joints
Joints:
- joint left_roll_joint: limit lower=-0.2 upper=0.5 effort=30 velocity=23 -> lower=-0.1 upper=0.5 effort=30 velocity=23
- joint left_yaw_joint: limit lower=-0.5 upper=0.5 effort=30 velocity=23 -> lower=-0.1 upper=0.1 effort=30 velocity=23
- joint right_roll_joint: limit lower=-0.5 upper=0.2 effort=30 velocity=23 -> lower=-0.5 upper=0.1 effort=30 velocity=23
- joint right_yaw_joint: limit lower=-0.3 upper=0.3 effort=30 velocity=23 -> lower=-0.1 upper=0.1 effort=30 velocity=23

Commit message: good

File: legged_train/resources/robots/wow/urdf/wow.urdf (robot description, URDF)
Before this commit: robot wow1, 11 links, 10 joints
Joints:
- joint left_roll_joint: limit lower=-0.1 upper=0.5 effort=30 velocity=23 -> lower=-0.1 upper=0.2 effort=30 velocity=23
- joint right_roll_joint: limit lower=-0.5 upper=0.1 effort=30 velocity=23 -> lower=-0.2 upper=0.1 effort=30 velocity=23
